File: Eagle/EMG.sch (EAGLE design)
At the start: 27 parts, among them IC1 AD623N, IC2 OPA344P, IC3 OPA344P, IC4 OPA344P, IC5 OPA344P, IC6 OPA344P, IC7 OPA344P

Commit message: Add files via upload
Parts:
- added IC9: MAX339CPE, maxim:MAX339CPE
- added PAD1, PAD10, PAD11, PAD12, PAD13, PAD14, PAD15, PAD16, PAD17, PAD2, PAD3, PAD4, PAD5, PAD6, PAD7, PAD8, PAD9: (no value), wirepad:1,6/0,8
Connections:
- removed net N$5: C1.1, C2.2
- new net N$20: IC1.-, IC9.COMA
- new net N$21: IC1.+, IC9.COMB
- new net N$22: IC9.NO4B, PAD11.P
- new net N$23: IC9.NO1A, PAD4.P
- new net N$24: IC9.NO2A, PAD5.P
- new net N$25: IC9.NO3A, PAD6.P
- new net N$26: IC9.NO4A, PAD7.P
- new net N$27: IC9.NO1B, PAD8.P
- new net N$28: IC9.NO3B, PAD10.P
- new net N$29: IC9.NO2B, PAD9.P
- new net N$30: IC9.A0, PAD12.P
- new net N$31: IC9.A1, PAD13.P
- new net N$32: IC9.EN, PAD14.P
- net +9V: now also IC9.V+, PAD3.P
- net -9V: now also IC9.V-, PAD1.P
- net GND: now also C1.1, C2.2, IC9.GND, PAD2.P
Other:
- moved on the sheet: C1

Commit message: Fixing Jerry's upload
Connections:
- net GND: now also PAD16.P, PAD17.P
- net N$16: now also PAD15.P
Other:
- moved on the sheet: PAD15
Changed lines of the file:
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@@
 <instance part="PAD13" gate="P" x="-1668.78" y="2.54"/>
 <instance part="PAD14" gate="P" x="-1668.78" y="0"/>
-<instance part="PAD15" gate="P" x="-1328.42" y="15.24"/>
+<instance part="PAD15" gate="P" x="-1328.42" y="15.24" rot="R180"/>
 <instance part="PAD16" gate="P" x="-1625.6" y="-27.94"/>
 <instance part="PAD17" gate="P" x="-1645.92" y="-27.94"/>
@@
 <wire x1="-1366.52" y1="12.7" x2="-1366.52" y2="-12.7" width="0.1524" layer="91"/>
 <wire x1="-1617.98" y1="-12.7" x2="-1623.06" y2="-12.7" width="0.1524" layer="91"/>
+<pinref part="IC9" gate="G$3" pin="GND"/>
 <wire x1="-1623.06" y1="-12.7" x2="-1643.38" y2="-12.7" width="0.1524" layer="91"/>
-<pinref part="IC9" gate="G$3" pin="GND"/>
 <wire x1="-1643.38" y1="-12.7" x2="-1663.7" y2="-12.7" width="0.1524" layer="91"/>
 <wire x1="-1663.7" y1="-12.7" x2="-1666.24" y2="-12.7" width="0.1524" layer="91"/>
@@
 <pinref part="PAD2" gate="P" pin="P"/>
 <junction x="-1663.7" y="-12.7"/>
-<wire x1="-1623.06" y1="-12.7" x2="-1623.06" y2="-27.94" width="0.1524" layer="91"/>
-<wire x1="-1643.38" y1="-12.7" x2="-1643.38" y2="-27.94" width="0.1524" layer="91"/>
-<junction x="-1643.38" y="-12.7"/>
 <pinref part="C1" gate="G$1" pin="1"/>
 <junction x="-1546.86" y="-12.7"/>
@@
 <wire x1="-1549.4" y1="-10.16" x2="-1549.4" y2="-12.7" width="0.1524" layer="91"/>
 <junction x="-1549.4" y="-12.7"/>
+<pinref part="PAD17" gate="P" pin="P"/>
+<wire x1="-1643.38" y1="-27.94" x2="-1643.38" y2="-12.7" width="0.1524" layer="91"/>
+<junction x="-1643.38" y="-12.7"/>
+<pinref part="PAD16" gate="P" pin="P"/>
+<wire x1="-1623.06" y1="-27.94" x2="-1623.06" y2="-12.7" width="0.1524" layer="91"/>
 </segment>
 </net>
@@
 <pinref part="R12" gate="G$1" pin="2"/>
 <wire x1="-1351.28" y1="30.48" x2="-1353.82" y2="30.48" width="0.1524" layer="91"/>
-<wire x1="-1351.28" y1="15.24" x2="-1328.42" y2="15.24" width="0.1524" layer="91"/>
+<pinref part="PAD15" gate="P" pin="P"/>
+<wire x1="-1351.28" y1="15.24" x2="-1330.96" y2="15.24" width="0.1524" layer="91"/>
 <junction x="-1351.28" y="15.24"/>
 </segment>

Commit message: Compressed brd
Parts:
- PAD1, PAD10, PAD11, PAD12, PAD13, PAD14, PAD15, PAD16, PAD17, PAD2, PAD3, PAD4, PAD5, PAD6, PAD7, PAD8, PAD9: device wirepad:1,6/0,8 -> wirepad:2,15/1,0
